Commit message: fixed GPS_link, incorrect file reference

File: husky_description/urdf/husky.urdf.xacro (robot description, xacro)
@@ -99,4 +99,11 @@
   <gazebo reference="imu_link">
   </gazebo>
+  <link name="GPS_link"/>
+  <joint name="GPS_joint" type="fixed">\
+    <origin xyz="$(optenv HUSKY_GPS_XYZ 0.19 0 0.149)" rpy="$(optenv HUSKY_GPS_RPY 0 -1.5708 3.1416)" />
+    <parent link="base_link" />
+    <child link="GPS_link" />
+  </joint>
+  <gazebo reference="GPS_link"></gazebo>
   <!-- Husky wheel macros -->
   <xacro:husky_wheel wheel_prefix="front_left">

Commit message: fixes, basic navigation working

File: husky_description/urdf/husky.urdf.xacro (robot description, xacro)
@@ -101,5 +101,5 @@
   <link name="GPS_link"/>
   <joint name="GPS_joint" type="fixed">\
-    <origin xyz="$(optenv HUSKY_GPS_XYZ 0.19 0 0.149)" rpy="$(optenv HUSKY_GPS_RPY 0 -1.5708 3.1416)" />
+    <origin xyz="$(optenv HUSKY_IMU_XYZ 0.19 0 0.149)" rpy="$(optenv HUSKY_IMU_RPY 0 -1.5708 3.1416)" />
     <parent link="base_link" />
     <child link="GPS_link" />
